Commit message: 有种吃屎的感觉

File: src/dingo/dingo_description/urdf/dingo.urdf.xacro (robot description, xacro)
@@ -1,8 +1,8 @@
 <?xml version="1.0"?>
 <robot name="dingo" xmlns:xacro="http://www.ros.org/wiki/xacro">
-  <xacro:if value="$(optenv DINGO_OMNI 0)">
+  <xacro:if value="$(optenv DINGO_OMNI 1)">
     <xacro:include filename="$(find dingo_description)/urdf/dingo-o.urdf.xacro" />
   </xacro:if>
-  <xacro:unless value="$(optenv DINGO_OMNI 0)">
+  <xacro:unless value="$(optenv DINGO_OMNI 1)">
     <xacro:include filename="$(find dingo_description)/urdf/dingo-d.urdf.xacro" />
   </xacro:unless>

File: src/dingo/dingo_description/urdf/pacs.urdf.xacro (robot description, xacro)
@@ -278,5 +278,5 @@
   <!-- Entire PACS System -->
   <xacro:macro name="pacs">
-    <xacro:property name="omni" value="$(optenv DINGO_OMNI 0)"/>
+    <xacro:property name="omni" value="$(optenv DINGO_OMNI 1)"/>
     <xacro:property name="riser" value="$(optenv DINGO_PACS_RISER 0)"/>
     <xacro:property name="pacs_enabled" value="$(optenv DINGO_PACS_ENABLED 0)" />

File: src/unidingo_description/urdf/uni_dingo_dual_arm.urdf.xacro (robot description, xacro)
@@ -24,4 +24,11 @@
   <!-- ========== Dingo 底盘（官方描述） ========== -->
   <xacro:include filename="$(find dingo_description)/urdf/dingo.urdf.xacro"/>
+  <!-- Enable self-collision for base links in Gazebo -->
+  <gazebo reference="base_link">
+    <self_collide>true</self_collide>
+  </gazebo>
+  <gazebo reference="chassis_link">
+    <self_collide>true</self_collide>
+  </gazebo>
   <!-- ========== 左臂安装座（仅作为连接点，不显示原有 mesh） ========== -->
   <link name="leftarm_link">

File: src/unidingo_description/urdf/z1_arm.urdf.xacro (robot description, xacro)
@@ -306,4 +306,26 @@
     <xacro:z1_motorTransmission prefix="${prefix}" name="5"/>
     <xacro:z1_motorTransmission prefix="${prefix}" name="6"/>
+    <!-- Enable self-collision in Gazebo for arm links -->
+    <gazebo reference="${prefix}link00">
+      <self_collide>true</self_collide>
+    </gazebo>
+    <gazebo reference="${prefix}link01">
+      <self_collide>true</self_collide>
+    </gazebo>
+    <gazebo reference="${prefix}link02">
+      <self_collide>true</self_collide>
+    </gazebo>
+    <gazebo reference="${prefix}link03">
+      <self_collide>true</self_collide>
+    </gazebo>
+    <gazebo reference="${prefix}link04">
+      <self_collide>true</self_collide>
+    </gazebo>
+    <gazebo reference="${prefix}link05">
+      <self_collide>true</self_collide>
+    </gazebo>
+    <gazebo reference="${prefix}link06">
+      <self_collide>true</self_collide>
+    </gazebo>
   </xacro:macro>
 </robot>
