Commit message: checkpoint-1021

File: src/dingo/dingo_description/urdf/dingo-d.urdf.xacro (robot description, xacro)
@@ -1,5 +1,4 @@
 <?xml version="1.0"?>
 <robot name="dingo" xmlns:xacro="http://www.ros.org/wiki/xacro">
-  <xacro:property name="pacs_enabled" value="$(optenv DINGO_PACS_ENABLED 0)"/>
   <xacro:property name="PI" value="3.1415926535897931" />
   <xacro:property name="wheel_radius" value="0.049" />
@@ -38,13 +37,4 @@
       </inertial>
     </link>
-    <gazebo reference="${prefix}_wheel_link">
-      <material>Gazebo/DarkGrey</material>
-      <selfCollide>false</selfCollide>
-      <mu1 value="0.5"/>
-      <mu2 value="0.5"/>
-      <kp value="10000000.0" />
-      <kd value="1" />
-      <fdir1 value="1 0 0"/>
-    </gazebo>
     <joint name="${prefix}_wheel" type="continuous">
       <parent link="chassis_link"/>
@@ -82,14 +72,4 @@
       </geometry>
       <origin rpy="0 0 0" xyz="0 0 0"/>
-      <surface>
-        <friction>
-          <ode>
-            <mu>0.0</mu>
-            <mu2>0.0</mu2>
-            <slip1>1.0</slip1>
-            <slip2>1.0</slip2>
-          </ode>
-        </friction>
-      </surface>
     </collision>
     <inertial>
@@ -106,14 +86,4 @@
     <origin xyz="-0.244 0 -0.00674" rpy="0 0 0"/>
   </joint>
-  <gazebo reference="rear_caster">
-    <turnGravityOff>false</turnGravityOff>
-    <kp>1000000.0</kp>
-    <kd>100.0</kd>
-    <mu1>0.2</mu1>
-    <mu2>0.2</mu2>
-    <fdir1>1 0 0</fdir1>
-    <minDepth>0.00</minDepth>
-    <implicitSpringDamper>1</implicitSpringDamper>
-  </gazebo>
   <link name="base_link"></link>
   <joint name="base_link_joint" type="fixed">
@@ -144,5 +114,5 @@
         iyy="0.2458" iyz="0"
         izz="0.4474"/>
-      </inertial>
+    </inertial>
   </link>
   <link name="imu_link">
@@ -157,16 +127,5 @@
     <child link="imu_link" />
   </joint>
-  <!--
-    Mounting points for accessories in the top channel.
-    These are flush with the top of the robot and all oriented to face forwards.
-    Dingo-D has 6 evenly-spaced 80mm mounts
-    We name the mounts (from front to back)
-      - front
-      - front b
-      - front c
-      - rear c
-      - rear b
-      - rear
-  -->
+  <!-- Mounting points for accessories in the top channel -->
   <link name="front_mount"/>
   <link name="front_b_mount"/>
@@ -205,9 +164,5 @@
     <child link="rear_mount" />
   </joint>
-  <!--
-    Mounting point for accessories on the front bumper.
-    Use with caution, but thin sensors (e.g Raspberry Pi NoIR camera) could
-    be mounted here for low-budget, front-facing capabilities
-  -->
+  <!-- Mounting point for accessories on the front bumper -->
   <link name="front_bumper_mount"></link>
   <joint name="front_bumper_mount_joint" type="fixed">
@@ -216,14 +171,3 @@
     <child link="front_bumper_mount" />
   </joint>
-  <!-- PACS -->
-  <xacro:include filename="$(find dingo_description)/urdf/pacs.urdf.xacro"/>
-  <xacro:pacs/>
-  <!-- Bring in simulation data for Gazebo. -->
-  <xacro:include filename="$(find dingo_description)/urdf/dingo.gazebo" />
-  <!-- Optional standard accessories, including their simulation data. The rendering
-       of these into the final description is controlled by optenv variables, which
-       default each one to off.-->
-  <xacro:include filename="$(find dingo_description)/urdf/accessories.urdf.xacro" />
-  <!-- Optional custom includes. -->
-  <xacro:include filename="$(optenv DINGO_URDF_EXTRAS empty.urdf)" />
 </robot>

File: src/dingo/dingo_description/urdf/dingo-o.urdf.xacro (robot description, xacro)
@@ -1,5 +1,4 @@
 <?xml version="1.0"?>
 <robot name="dingo" xmlns:xacro="http://www.ros.org/wiki/xacro">
-  <xacro:property name="pacs_enabled" value="$(optenv DINGO_PACS_ENABLED 0)" />
   <xacro:property name="PI" value="3.1415926535897931" />
   <xacro:property name="wheelbase" value="0.570" />
@@ -95,5 +94,5 @@
         iyy="0.7266" iyz="0"
         izz="1.0553"/>
-      </inertial>
+    </inertial>
   </link>
   <link name="imu_link">
@@ -108,17 +107,5 @@
     <child link="imu_link" />
   </joint>
-  <!--
-    Mounting points for accessories in the top channel.
-    These are flush with the top of the robot and all oriented to face forwards.
-    Dingo-D has 6 evenly-spaced 80mm mounts
-    We name the mounts (from front to back)
-      - front
-      - front b
-      - front c
-      - mid
-      - rear c
-      - rear b
-      - rear
-  -->
+  <!-- Mounting points for accessories in the top channel -->
   <link name="front_mount"/>
   <link name="front_b_mount"/>
@@ -163,9 +150,5 @@
     <child link="rear_mount" />
   </joint>
-  <!--
-    Mounting point for accessories on the front bumper.
-    Use with caution, but thin sensors (e.g Raspberry Pi NoIR camera) could
-    be mounted here for low-budget, front/rear-facing capabilities
-  -->
+  <!-- Mounting point for accessories on the front bumper -->
   <link name="front_bumper_mount"></link>
   <joint name="front_bumper_mount_joint" type="fixed">
@@ -174,15 +157,3 @@
     <child link="front_bumper_mount" />
   </joint>
-  <!-- PACS -->
-  <xacro:include filename="$(find dingo_description)/urdf/pacs.urdf.xacro"/>
-  <xacro:pacs/>
-  <!-- Bring in simulation data for Gazebo. -->
-  <xacro:include filename="$(find dingo_description)/urdf/dingo.gazebo" />
-  <xacro:include filename="$(find dingo_description)/urdf/dingo-o.gazebo" />
-  <!-- Optional standard accessories, including their simulation data. The rendering
-       of these into the final description is controlled by optenv variables, which
-       default each one to off.-->
-  <xacro:include filename="$(find dingo_description)/urdf/accessories.urdf.xacro" />
-  <!-- Optional custom includes. -->
-  <xacro:include filename="$(optenv DINGO_URDF_EXTRAS empty.urdf)" />
 </robot>

File: src/dingo/dingo_description/urdf/dingo.urdf.xacro (robot description, xacro)
@@ -1,8 +1,9 @@
 <?xml version="1.0"?>
 <robot name="dingo" xmlns:xacro="http://www.ros.org/wiki/xacro">
-  <xacro:if value="$(optenv DINGO_OMNI 1)">
+  <xacro:arg name="dingo_omni" default="$(optenv DINGO_OMNI 1)" />
+  <xacro:if value="$(arg dingo_omni)">
     <xacro:include filename="$(find dingo_description)/urdf/dingo-o.urdf.xacro" />
   </xacro:if>
-  <xacro:unless value="$(optenv DINGO_OMNI 1)">
+  <xacro:unless value="$(arg dingo_omni)">
     <xacro:include filename="$(find dingo_description)/urdf/dingo-d.urdf.xacro" />
   </xacro:unless>
