Commit message: 未完成

File: src/dingo/dingo_description/urdf/accessories/intel_realsense.urdf.xacro (robot description, xacro)
@@ -85,6 +85,6 @@
              <width>${width}</width>
              <height>${height}</height>
-             <!-- TODO: check what format the Realsense hardware delivers and set this to match! -->
-             <format>RGB8</format>
+             <!-- Gazebo supported format: R8G8B8 -->
+             <format>R8G8B8</format>
            </image>
            <clip>

File: src/unidingo_description/urdf/uni_dingo_dual_arm.urdf.xacro (robot description, xacro)
@@ -53,5 +53,5 @@
     <child link="leftarm_link"/>
   </joint>
-  <!-- ========== 左臂支撑柱（仅视觉） ========== -->
+  <!-- ========== 左臂支撑柱 ========== -->
   <link name="leftarm_support_link">
     <visual>
@@ -62,4 +62,10 @@
       <material name="arm_support_grey"/>
     </visual>
+    <collision>
+      <origin xyz="0 0 ${-left_arm_support_length/2.0}" rpy="0 0 0"/>
+      <geometry>
+        <cylinder length="${left_arm_support_length}" radius="${arm_support_radius}"/>
+      </geometry>
+    </collision>
   </link>
   <joint name="base_leftarm_support_joint" type="fixed">
@@ -82,5 +88,5 @@
     <child link="rightarm_link"/>
   </joint>
-  <!-- ========== 右臂支撑柱（仅视觉） ========== -->
+  <!-- ========== 右臂支撑柱 ========== -->
   <link name="rightarm_support_link">
     <visual>
@@ -91,4 +97,10 @@
       <material name="arm_support_grey"/>
     </visual>
+    <collision>
+      <origin xyz="0 0 ${-right_arm_support_length/2.0}" rpy="0 0 0"/>
+      <geometry>
+        <cylinder length="${right_arm_support_length}" radius="${arm_support_radius}"/>
+      </geometry>
+    </collision>
   </link>
   <joint name="base_rightarm_support_joint" type="fixed">
@@ -107,5 +119,5 @@
   <!-- ========== Pan-Tilt 云台 ========== -->
   <xacro:if value="$(arg PanTilt)">
-    <!-- 云台支撑柱（仅视觉） -->
+    <!-- 云台支撑柱 -->
     <link name="pan_tilt_support_link">
       <visual>
@@ -116,4 +128,10 @@
         <material name="arm_support_grey"/>
       </visual>
+      <collision>
+        <origin xyz="0 0 ${-pan_tilt_support_length/2.0}" rpy="0 0 0"/>
+        <geometry>
+          <cylinder length="${pan_tilt_support_length}" radius="${arm_support_radius}"/>
+        </geometry>
+      </collision>
     </link>
     <joint name="base_pan_tilt_support_joint" type="fixed">
@@ -126,5 +144,5 @@
       <origin xyz="${pan_tilt_mount_x} ${pan_tilt_mount_y} ${pan_tilt_mount_z}" rpy="0 0 0"/>
     </xacro:pan_tilt>
-    <!-- 相机支撑柱（仅视觉） -->
+    <!-- 相机支撑柱 -->
     <xacro:property name="camera_mount_z" value="0.1"/>
     <link name="camera_support_link">
@@ -136,4 +154,10 @@
         <material name="arm_support_grey"/>
       </visual>
+      <collision>
+        <origin xyz="0 0 ${camera_mount_z/2.0}" rpy="0 0 0"/>
+        <geometry>
+          <cylinder length="${camera_mount_z}" radius="${arm_support_radius}"/>
+        </geometry>
+      </collision>
     </link>
     <joint name="pan_tilt_camera_support_joint" type="fixed">

File: src/unidingo_description/urdf/z1_arm.urdf.xacro (robot description, xacro)
@@ -71,4 +71,10 @@
         </geometry>
       </visual>
+      <collision>
+        <origin rpy="0 0 0" xyz="0 0 0"/>
+        <geometry>
+          <mesh filename="package://z1_description/meshes/collision/z1_Link01.STL" scale="1 1 1"/>
+        </geometry>
+      </collision>
       <inertial>
         <origin rpy="0 0 0" xyz="${L01_ComX} ${L01_ComY} ${L01_ComZ}"/>
@@ -203,4 +209,10 @@
         </geometry>
       </visual>
+      <collision>
+        <origin rpy="0 0 0" xyz="0 0 0"/>
+        <geometry>
+          <mesh filename="package://z1_description/meshes/collision/z1_Link05.STL" scale="1 1 1"/>
+        </geometry>
+      </collision>
       <inertial>
         <origin rpy="0 0 0" xyz="${L05_ComX} ${L05_ComY} ${L05_ComZ}"/>
