Commit message: 可以用键盘和rviz控制机械臂

File: src/unidingo_description/urdf/uni_dingo_dual_arm.urdf.xacro (robot description, xacro)
@@ -7,30 +7,21 @@
   <!-- 参数 -->
   <xacro:arg name="UnitreeGripper" default="true"/>
+  <xacro:property name="arm_support_radius" value="0.02"/>
+  <xacro:property name="arm_support_clearance" value="0.10"/>
+  <xacro:property name="left_arm_mount_x" value="0.15091"/>
+  <xacro:property name="left_arm_mount_y" value="-0.11708"/>
+  <xacro:property name="left_arm_mount_z" value="0.57228"/>
+  <xacro:property name="left_arm_support_length" value="${left_arm_mount_z - arm_support_clearance}"/>
+  <xacro:property name="right_arm_mount_x" value="0.15091"/>
+  <xacro:property name="right_arm_mount_y" value="0.11708"/>
+  <xacro:property name="right_arm_mount_z" value="0.57228"/>
+  <xacro:property name="right_arm_support_length" value="${right_arm_mount_z - arm_support_clearance}"/>
+  <material name="arm_support_grey">
+    <color rgba="0.3 0.3 0.3 1.0"/>
+  </material>
   <!-- 引入 Z1 机械臂 macro -->
   <xacro:include filename="$(find uni_dingo)/urdf/z1_arm.urdf.xacro"/>
-  <!-- ========== Dingo 底盘 ========== -->
-  <link name="base_link">
-    <inertial>
-      <origin xyz="-0.022862 -0.034436 0.035407" rpy="0 0 0"/>
-      <mass value="5.3306"/>
-      <inertia ixx="0.059795" ixy="2.6827E-06" ixz="-1.8684E-07"
-               iyy="0.020279" iyz="0.00018072" izz="0.06071"/>
-    </inertial>
-    <visual>
-      <origin xyz="0 0 0" rpy="0 0 0"/>
-      <geometry>
-        <mesh filename="package://uni_dingo/meshes/base_link.STL"/>
-      </geometry>
-      <material name="">
-        <color rgba="1 1 1 1"/>
-      </material>
-    </visual>
-    <collision>
-      <origin xyz="0 0 0" rpy="0 0 0"/>
-      <geometry>
-        <mesh filename="package://uni_dingo/meshes/base_link.STL"/>
-      </geometry>
-    </collision>
-  </link>
+  <!-- ========== Dingo 底盘（官方描述） ========== -->
+  <xacro:include filename="$(find dingo_description)/urdf/dingo.urdf.xacro"/>
   <!-- ========== 左臂安装座（仅作为连接点，不显示原有 mesh） ========== -->
   <link name="leftarm_link">
@@ -43,7 +34,22 @@
   </link>
   <joint name="base_leftarm_joint" type="fixed">
-    <origin xyz="0.11708 -0.15091 0.57228" rpy="0 0 0"/>
+    <origin xyz="${left_arm_mount_x} ${left_arm_mount_y} ${left_arm_mount_z}" rpy="0 0 0"/>
     <parent link="base_link"/>
     <child link="leftarm_link"/>
+  </joint>
+  <!-- ========== 左臂支撑柱（仅视觉） ========== -->
+  <link name="leftarm_support_link">
+    <visual>
+      <origin xyz="0 0 ${-left_arm_support_length/2.0}" rpy="0 0 0"/>
+      <geometry>
+        <cylinder length="${left_arm_support_length}" radius="${arm_support_radius}"/>
+      </geometry>
+      <material name="arm_support_grey"/>
+    </visual>
+  </link>
+  <joint name="base_leftarm_support_joint" type="fixed">
+    <origin xyz="${left_arm_mount_x} ${left_arm_mount_y} ${left_arm_mount_z}" rpy="0 0 0"/>
+    <parent link="base_link"/>
+    <child link="leftarm_support_link"/>
   </joint>
   <!-- ========== 右臂安装座（仅作为连接点，不显示原有 mesh） ========== -->
@@ -57,15 +63,30 @@
   </link>
   <joint name="base_rightarm_joint" type="fixed">
-    <origin xyz="-0.11708 -0.15091 0.57228" rpy="0 0 0"/>
+    <origin xyz="${right_arm_mount_x} ${right_arm_mount_y} ${right_arm_mount_z}" rpy="0 0 0"/>
     <parent link="base_link"/>
     <child link="rightarm_link"/>
   </joint>
-  <!-- ========== 左 Z1 机械臂（朝前，绕 Z 轴旋转 -90°） ========== -->
+  <!-- ========== 右臂支撑柱（仅视觉） ========== -->
+  <link name="rightarm_support_link">
+    <visual>
+      <origin xyz="0 0 ${-right_arm_support_length/2.0}" rpy="0 0 0"/>
+      <geometry>
+        <cylinder length="${right_arm_support_length}" radius="${arm_support_radius}"/>
+      </geometry>
+      <material name="arm_support_grey"/>
+    </visual>
+  </link>
+  <joint name="base_rightarm_support_joint" type="fixed">
+    <origin xyz="${right_arm_mount_x} ${right_arm_mount_y} ${right_arm_mount_z}" rpy="0 0 0"/>
+    <parent link="base_link"/>
+    <child link="rightarm_support_link"/>
+  </joint>
+  <!-- ========== 左 Z1 机械臂 ========== -->
   <xacro:z1_arm prefix="left_" parent="leftarm_link" UnitreeGripper="$(arg UnitreeGripper)">
-    <origin xyz="0 0 0" rpy="0 0 ${-pi/2}"/>
+    <origin xyz="0 0 0" rpy="0 0 0"/>
   </xacro:z1_arm>
-  <!-- ========== 右 Z1 机械臂（朝前，绕 Z 轴旋转 -90°） ========== -->
+  <!-- ========== 右 Z1 机械臂 ========== -->
   <xacro:z1_arm prefix="right_" parent="rightarm_link" UnitreeGripper="$(arg UnitreeGripper)">
-    <origin xyz="0 0 0" rpy="0 0 ${-pi/2}"/>
+    <origin xyz="0 0 0" rpy="0 0 0"/>
   </xacro:z1_arm>
 </robot>

Commit message: model description

File: src/unidingo_description/urdf/uni_dingo_dual_arm.urdf.xacro (robot description, xacro)
@@ -2,10 +2,16 @@
 <!--
   Uni-Dingo 双臂机器人描述
-  包含: Dingo 底盘 + 左 Z1 机械臂 + 右 Z1 机械臂
+  包含: Dingo 底盘 + 左 Z1 机械臂 + 右 Z1 机械臂 + Pan-Tilt 云台
 -->
 <robot name="uni_dingo_dual_arm" xmlns:xacro="http://www.ros.org/wiki/xacro">
   <!-- 参数 -->
   <xacro:arg name="UnitreeGripper" default="true"/>
+  <xacro:arg name="PanTilt" default="true"/>
   <xacro:property name="arm_support_radius" value="0.02"/>
+  <!-- 云台挂载位置 -->
+  <xacro:property name="pan_tilt_mount_x" value="0.15091"/>
+  <xacro:property name="pan_tilt_mount_y" value="0"/>
+  <xacro:property name="pan_tilt_mount_z" value="1.0"/>
+  <xacro:property name="pan_tilt_support_length" value="${pan_tilt_mount_z - arm_support_clearance}"/>
   <xacro:property name="arm_support_clearance" value="0.10"/>
   <xacro:property name="left_arm_mount_x" value="0.15091"/>
@@ -22,4 +28,6 @@
   <!-- 引入 Z1 机械臂 macro -->
   <xacro:include filename="$(find uni_dingo)/urdf/z1_arm.urdf.xacro"/>
+  <!-- 引入 Pan-Tilt 云台 macro -->
+  <xacro:include filename="$(find pan_tilt_description)/urdf/pan_tilt.urdf.xacro"/>
   <!-- ========== Dingo 底盘（官方描述） ========== -->
   <xacro:include filename="$(find dingo_description)/urdf/dingo.urdf.xacro"/>
@@ -97,3 +105,49 @@
     <origin xyz="0 0 0" rpy="0 0 0"/>
   </xacro:z1_arm>
+  <!-- ========== Pan-Tilt 云台 ========== -->
+  <xacro:if value="$(arg PanTilt)">
+    <!-- 云台支撑柱（仅视觉） -->
+    <link name="pan_tilt_support_link">
+      <visual>
+        <origin xyz="0 0 ${-pan_tilt_support_length/2.0}" rpy="0 0 0"/>
+        <geometry>
+          <cylinder length="${pan_tilt_support_length}" radius="${arm_support_radius}"/>
+        </geometry>
+        <material name="arm_support_grey"/>
+      </visual>
+    </link>
+    <joint name="base_pan_tilt_support_joint" type="fixed">
+      <origin xyz="${pan_tilt_mount_x} ${pan_tilt_mount_y} ${pan_tilt_mount_z}" rpy="0 0 0"/>
+      <parent link="base_link"/>
+      <child link="pan_tilt_support_link"/>
+    </joint>
+    <!-- 云台 -->
+    <xacro:pan_tilt parent="base_link">
+      <origin xyz="${pan_tilt_mount_x} ${pan_tilt_mount_y} ${pan_tilt_mount_z}" rpy="0 0 0"/>
+    </xacro:pan_tilt>
+    <!-- 相机支撑柱（仅视觉） -->
+    <xacro:property name="camera_mount_z" value="0.1"/>
+    <link name="camera_support_link">
+      <visual>
+        <origin xyz="0 0 ${camera_mount_z/2.0}" rpy="0 0 0"/>
+        <geometry>
+          <cylinder length="${camera_mount_z}" radius="${arm_support_radius}"/>
+        </geometry>
+        <material name="arm_support_grey"/>
+      </visual>
+    </link>
+    <joint name="pan_tilt_camera_support_joint" type="fixed">
+      <origin xyz="0 0 0" rpy="0 0 0"/>
+      <parent link="pan_tilt_surface"/>
+      <child link="camera_support_link"/>
+    </joint>
+    <!-- D455 相机（挂载到云台顶部，z 方向偏移 0.1m） -->
+    <xacro:realsense_sensor rs_model="d455"
+                            prefix="head"
+                            parent="pan_tilt_surface"
+                            topic="d455"
+                            include="0">
+      <origin xyz="0 0 ${camera_mount_z}" rpy="0 0 0"/>
+    </xacro:realsense_sensor>
+  </xacro:if>
 </robot>

Commit message: 真机成功

File: src/unidingo_description/urdf/uni_dingo_dual_arm.urdf.xacro (robot description, xacro)
@@ -16,9 +16,9 @@
   <xacro:property name="arm_support_clearance" value="0.10"/>
   <xacro:property name="left_arm_mount_x" value="0.15091"/>
-  <xacro:property name="left_arm_mount_y" value="-0.11708"/>
+  <xacro:property name="left_arm_mount_y" value="0.11708"/>
   <xacro:property name="left_arm_mount_z" value="0.57228"/>
   <xacro:property name="left_arm_support_length" value="${left_arm_mount_z - arm_support_clearance}"/>
   <xacro:property name="right_arm_mount_x" value="0.15091"/>
-  <xacro:property name="right_arm_mount_y" value="0.11708"/>
+  <xacro:property name="right_arm_mount_y" value="-0.11708"/>
   <xacro:property name="right_arm_mount_z" value="0.57228"/>
   <xacro:property name="right_arm_support_length" value="${right_arm_mount_z - arm_support_clearance}"/>
