Commit message: 双臂测试文件

File: src/unidingo_description/urdf/uni_dingo_dual_arm.urdf.xacro (robot description, xacro)
@@ -30,4 +30,5 @@
   <!-- 引入 Pan-Tilt 云台 macro -->
   <xacro:include filename="$(find pan_tilt_description)/urdf/pan_tilt.urdf.xacro"/>
+  <xacro:include filename="$(find uni_dingo)/urdf/d455_visual.urdf.xacro"/>
   <!-- ========== Dingo 底盘（官方描述） ========== -->
   <xacro:include filename="$(find dingo_description)/urdf/dingo.urdf.xacro"/>
@@ -174,11 +175,7 @@
     </joint>
     <!-- D455 相机（挂载到相机支撑柱顶端） -->
-    <xacro:realsense_sensor rs_model="d455"
-                            prefix="head"
-                            parent="camera_support_link"
-                            topic="d455"
-                            include="0">
+    <xacro:d455_visual parent="camera_support_link">
       <origin xyz="0 0 ${camera_mount_z}" rpy="0 0 0"/>
-    </xacro:realsense_sensor>
+    </xacro:d455_visual>
   </xacro:if>
 </robot>

File: src/unidingo_description/urdf/z1_arm.urdf.xacro (robot description, xacro)
@@ -252,4 +252,11 @@
       </inertial>
     </link>
+    <!-- Match z1_control.urdf: TCP is fixed, not the moving gripper finger. -->
+    <link name="${prefix}tool"/>
+    <joint name="${prefix}tool_mount" type="fixed">
+      <parent link="${prefix}link06"/>
+      <child link="${prefix}tool"/>
+      <origin xyz="0.051 0 0" rpy="0 0 0"/>
+    </joint>
     <!-- Unitree Gripper (可选) -->
     <xacro:if value="${UnitreeGripper}">
