Commit message: 部分精简

File: src/uni_dingo_api/urdf/sensors.gazebo.xacro (robot description, xacro)
@@ -5,5 +5,6 @@
   Include this file in your robot URDF to add:
   - RGB-D Camera (simulating Intel RealSense D455)
-  - Pan-Tilt head controllers
+  Note: Pan-Tilt transmissions and controllers are defined in
+  pan_tilt_description/urdf/pan_tilt.urdf.xacro, not here.
   Usage:
     <xacro:include filename="$(find uni_dingo_api)/urdf/sensors.gazebo.xacro"/>
@@ -102,32 +103,4 @@
       </sensor>
     </gazebo>
-    <!-- ==================== Pan-Tilt Controllers ==================== -->
-    <!-- Pan (Yaw) Controller -->
-    <transmission name="pan_tilt_yaw_trans">
-      <type>transmission_interface/SimpleTransmission</type>
-      <joint name="pan_tilt_yaw_joint">
-        <hardwareInterface>hardware_interface/PositionJointInterface</hardwareInterface>
-      </joint>
-      <actuator name="pan_tilt_yaw_motor">
-        <mechanicalReduction>1</mechanicalReduction>
-      </actuator>
-    </transmission>
-    <!-- Tilt (Pitch) Controller -->
-    <transmission name="pan_tilt_pitch_trans">
-      <type>transmission_interface/SimpleTransmission</type>
-      <joint name="pan_tilt_pitch_joint">
-        <hardwareInterface>hardware_interface/PositionJointInterface</hardwareInterface>
-      </joint>
-      <actuator name="pan_tilt_pitch_motor">
-        <mechanicalReduction>1</mechanicalReduction>
-      </actuator>
-    </transmission>
-    <!-- Gazebo ros_control plugin for pan-tilt -->
-    <gazebo>
-      <plugin name="pan_tilt_gazebo_ros_control" filename="libgazebo_ros_control.so">
-        <robotNamespace>/pan_tilt</robotNamespace>
-        <robotSimType>gazebo_ros_control/DefaultRobotHWSim</robotSimType>
-      </plugin>
-    </gazebo>
-  </xacro:macro>
+</xacro:macro>
 </robot>

File: src/unidingo_description/urdf/uni_dingo_dual_arm.urdf.xacro (robot description, xacro)
@@ -39,20 +39,18 @@
     <self_collide>true</self_collide>
   </gazebo>
-  <!-- ========== 左臂安装座（仅作为连接点，不显示原有 mesh） ========== -->
+  <!-- 支撑柱惯性参数（铝制圆柱，密度约 2700 kg/m³） -->
+  <xacro:property name="arm_support_mass" value="1.4"/>
+  <xacro:property name="pan_tilt_support_mass" value="2.7"/>
+  <!-- ========== 左臂安装座 + 支撑柱（合并为一个 link） ========== -->
   <link name="leftarm_link">
     <inertial>
-      <origin xyz="0 0 0" rpy="0 0 0"/>
-      <mass value="0.1"/>
-      <inertia ixx="0.001" ixy="0" ixz="0" iyy="0.001" iyz="0" izz="0.001"/>
+      <origin xyz="0 0 ${-left_arm_support_length/2.0}" rpy="0 0 0"/>
+      <mass value="${arm_support_mass}"/>
+      <inertia ixx="${arm_support_mass*(3*arm_support_radius*arm_support_radius + left_arm_support_length*left_arm_support_length)/12.0}"
+               ixy="0" ixz="0"
+               iyy="${arm_support_mass*(3*arm_support_radius*arm_support_radius + left_arm_support_length*left_arm_support_length)/12.0}"
+               iyz="0"
+               izz="${arm_support_mass*arm_support_radius*arm_support_radius/2.0}"/>
     </inertial>
-    <!-- 移除 visual，避免与 Z1 机械臂重复 -->
-  </link>
-  <joint name="base_leftarm_joint" type="fixed">
-    <origin xyz="${left_arm_mount_x} ${left_arm_mount_y} ${left_arm_mount_z}" rpy="0 0 0"/>
-    <parent link="base_link"/>
-    <child link="leftarm_link"/>
-  </joint>
-  <!-- ========== 左臂支撑柱 ========== -->
-  <link name="leftarm_support_link">
     <visual>
       <origin xyz="0 0 ${-left_arm_support_length/2.0}" rpy="0 0 0"/>
@@ -69,25 +67,20 @@
     </collision>
   </link>
-  <joint name="base_leftarm_support_joint" type="fixed">
+  <joint name="base_leftarm_joint" type="fixed">
     <origin xyz="${left_arm_mount_x} ${left_arm_mount_y} ${left_arm_mount_z}" rpy="0 0 0"/>
     <parent link="base_link"/>
-    <child link="leftarm_support_link"/>
+    <child link="leftarm_link"/>
   </joint>
-  <!-- ========== 右臂安装座（仅作为连接点，不显示原有 mesh） ========== -->
+  <!-- ========== 右臂安装座 + 支撑柱（合并为一个 link） ========== -->
   <link name="rightarm_link">
     <inertial>
-      <origin xyz="0 0 0" rpy="0 0 0"/>
-      <mass value="0.1"/>
-      <inertia ixx="0.001" ixy="0" ixz="0" iyy="0.001" iyz="0" izz="0.001"/>
+      <origin xyz="0 0 ${-right_arm_support_length/2.0}" rpy="0 0 0"/>
+      <mass value="${arm_support_mass}"/>
+      <inertia ixx="${arm_support_mass*(3*arm_support_radius*arm_support_radius + right_arm_support_length*right_arm_support_length)/12.0}"
+               ixy="0" ixz="0"
+               iyy="${arm_support_mass*(3*arm_support_radius*arm_support_radius + right_arm_support_length*right_arm_support_length)/12.0}"
+               iyz="0"
+               izz="${arm_support_mass*arm_support_radius*arm_support_radius/2.0}"/>
     </inertial>
-    <!-- 移除 visual，避免与 Z1 机械臂重复 -->
-  </link>
-  <joint name="base_rightarm_joint" type="fixed">
-    <origin xyz="${right_arm_mount_x} ${right_arm_mount_y} ${right_arm_mount_z}" rpy="0 0 0"/>
-    <parent link="base_link"/>
-    <child link="rightarm_link"/>
-  </joint>
-  <!-- ========== 右臂支撑柱 ========== -->
-  <link name="rightarm_support_link">
     <visual>
       <origin xyz="0 0 ${-right_arm_support_length/2.0}" rpy="0 0 0"/>
@@ -104,8 +97,8 @@
     </collision>
   </link>
-  <joint name="base_rightarm_support_joint" type="fixed">
+  <joint name="base_rightarm_joint" type="fixed">
     <origin xyz="${right_arm_mount_x} ${right_arm_mount_y} ${right_arm_mount_z}" rpy="0 0 0"/>
     <parent link="base_link"/>
-    <child link="rightarm_support_link"/>
+    <child link="rightarm_link"/>
   </joint>
   <!-- ========== 左 Z1 机械臂 ========== -->
@@ -119,6 +112,15 @@
   <!-- ========== Pan-Tilt 云台 ========== -->
   <xacro:if value="$(arg PanTilt)">
-    <!-- 云台支撑柱 -->
-    <link name="pan_tilt_support_link">
+    <!-- 云台安装座 + 支撑柱（合并为一个 link，云台挂载到此 link） -->
+    <link name="pan_tilt_mount_link">
+      <inertial>
+        <origin xyz="0 0 ${-pan_tilt_support_length/2.0}" rpy="0 0 0"/>
+        <mass value="${pan_tilt_support_mass}"/>
+        <inertia ixx="${pan_tilt_support_mass*(3*arm_support_radius*arm_support_radius + pan_tilt_support_length*pan_tilt_support_length)/12.0}"
+                 ixy="0" ixz="0"
+                 iyy="${pan_tilt_support_mass*(3*arm_support_radius*arm_support_radius + pan_tilt_support_length*pan_tilt_support_length)/12.0}"
+                 iyz="0"
+                 izz="${pan_tilt_support_mass*arm_support_radius*arm_support_radius/2.0}"/>
+      </inertial>
       <visual>
         <origin xyz="0 0 ${-pan_tilt_support_length/2.0}" rpy="0 0 0"/>
@@ -135,16 +137,21 @@
       </collision>
     </link>
-    <joint name="base_pan_tilt_support_joint" type="fixed">
+    <joint name="base_pan_tilt_mount_joint" type="fixed">
       <origin xyz="${pan_tilt_mount_x} ${pan_tilt_mount_y} ${pan_tilt_mount_z}" rpy="0 0 0"/>
       <parent link="base_link"/>
-      <child link="pan_tilt_support_link"/>
+      <child link="pan_tilt_mount_link"/>
     </joint>
-    <!-- 云台 -->
-    <xacro:pan_tilt parent="base_link">
-      <origin xyz="${pan_tilt_mount_x} ${pan_tilt_mount_y} ${pan_tilt_mount_z}" rpy="0 0 0"/>
+    <!-- 云台（挂载到支撑柱顶端） -->
+    <xacro:pan_tilt parent="pan_tilt_mount_link">
+      <origin xyz="0 0 0" rpy="0 0 0"/>
     </xacro:pan_tilt>
     <!-- 相机支撑柱 -->
     <xacro:property name="camera_mount_z" value="0.1"/>
     <link name="camera_support_link">
+      <inertial>
+        <origin xyz="0 0 ${camera_mount_z/2.0}" rpy="0 0 0"/>
+        <mass value="0.05"/>
+        <inertia ixx="0.00005" ixy="0" ixz="0" iyy="0.00005" iyz="0" izz="0.00001"/>
+      </inertial>
       <visual>
         <origin xyz="0 0 ${camera_mount_z/2.0}" rpy="0 0 0"/>
@@ -166,8 +173,8 @@
       <child link="camera_support_link"/>
     </joint>
-    <!-- D455 相机（挂载到云台顶部，z 方向偏移 0.1m） -->
+    <!-- D455 相机（挂载到相机支撑柱顶端） -->
     <xacro:realsense_sensor rs_model="d455"
                             prefix="head"
-                            parent="pan_tilt_surface"
+                            parent="camera_support_link"
                             topic="d455"
                             include="0">
