Commit message: 大提交

File: src/unidingo_description_ros2/urdf/dingo_base.xacro (robot description, xacro)
@@ -1,11 +1,12 @@
 <?xml version="1.0"?>
-<!--
-  Simplified Dingo base frame.
-  This provides the base_link and base_footprint for the Uni-Dingo robot.
-  In production, replace with official clearpath_common Dingo description.
-  Approximate dimensions: 0.52 x 0.38 x 0.15 m (Dingo-O omni platform)
--->
+<!-- Dingo omni base geometry for ROS2 simulation. -->
 <robot xmlns:xacro="http://www.ros.org/wiki/xacro">
     <xacro:macro name="dingo_base">
+        <xacro:property name="wheelbase" value="0.570"/>
+        <xacro:property name="track" value="0.3708"/>
+        <xacro:property name="wheel_vertical_offset" value="0.035145"/>
+        <xacro:property name="wheel_radius" value="0.050"/>
+        <xacro:property name="wheel_width" value="0.050"/>
+        <xacro:property name="wheel_mass" value="0.4"/>
         <link name="base_footprint"/>
         <joint name="base_footprint_joint" type="fixed">
@@ -14,11 +15,17 @@
             <child link="base_link"/>
         </joint>
-        <link name="base_link">
+        <link name="base_link"/>
+        <joint name="base_link_joint" type="fixed">
+            <origin xyz="0 0 0" rpy="0 0 0"/>
+            <parent link="base_link"/>
+            <child link="chassis_link"/>
+        </joint>
+        <link name="chassis_link">
             <inertial>
                 <origin xyz="0 0 0" rpy="0 0 0"/>
-                <mass value="15.0"/>
-                <inertia ixx="0.23" ixy="0" ixz="0"
-                         iyy="0.36" iyz="0"
-                         izz="0.52"/>
+                <mass value="14.0"/>
+                <inertia ixx="0.35498" ixy="0" ixz="0"
+                         iyy="0.7266" iyz="0"
+                         izz="1.0553"/>
             </inertial>
             <visual>
@@ -38,9 +45,49 @@
             </collision>
         </link>
+        <xacro:macro name="dingo_wheel" params="joint_name link_name x y">
+            <link name="${link_name}">
+                <inertial>
+                    <origin xyz="0 0 0" rpy="0 0 0"/>
+                    <mass value="${wheel_mass}"/>
+                    <inertia ixx="0.0003234" ixy="0" ixz="0"
+                             iyy="0.0003234" iyz="0"
+                             izz="0.0004901"/>
+                </inertial>
+                <visual>
+                    <origin xyz="0 0 0" rpy="1.5707963 0 0"/>
+                    <geometry>
+                        <cylinder radius="${wheel_radius}" length="${wheel_width}"/>
+                    </geometry>
+                    <material name="wheel_black">
+                        <color rgba="0.1 0.1 0.1 1.0"/>
+                    </material>
+                </visual>
+                <collision>
+                    <origin xyz="0 0 0" rpy="1.5707963 0 0"/>
+                    <geometry>
+                        <cylinder radius="${wheel_radius}" length="${wheel_width}"/>
+                    </geometry>
+                </collision>
+            </link>
+            <joint name="${joint_name}" type="continuous">
+                <origin xyz="${x} ${y} ${wheel_vertical_offset}" rpy="0 0 0"/>
+                <parent link="chassis_link"/>
+                <child link="${link_name}"/>
+                <axis xyz="0 1 0"/>
+            </joint>
+        </xacro:macro>
+        <xacro:dingo_wheel joint_name="front_left_wheel" link_name="front_left_wheel_link"
+                           x="${wheelbase/2.0}" y="${track/2.0 + wheel_width/2.0}"/>
+        <xacro:dingo_wheel joint_name="front_right_wheel" link_name="front_right_wheel_link"
+                           x="${wheelbase/2.0}" y="${-track/2.0 - wheel_width/2.0}"/>
+        <xacro:dingo_wheel joint_name="rear_left_wheel" link_name="rear_left_wheel_link"
+                           x="${-wheelbase/2.0}" y="${track/2.0 + wheel_width/2.0}"/>
+        <xacro:dingo_wheel joint_name="rear_right_wheel" link_name="rear_right_wheel_link"
+                           x="${-wheelbase/2.0}" y="${-track/2.0 - wheel_width/2.0}"/>
         <!-- IMU frame (for sensor integration) -->
         <link name="imu_link"/>
         <joint name="imu_joint" type="fixed">
             <origin xyz="0 0 0.075" rpy="0 0 0"/>
-            <parent link="base_link"/>
+            <parent link="chassis_link"/>
             <child link="imu_link"/>
         </joint>

File: src/unidingo_description_ros2/urdf/uni_dingo_dual_arm.urdf.xacro (robot description, xacro)
@@ -8,12 +8,18 @@
     <xacro:arg name="has_gripper" default="true"/>
     <xacro:arg name="pan_tilt" default="true"/>
-    <xacro:arg name="left_controller_ip" default="127.0.0.1"/>
-    <xacro:arg name="left_sdk_port" default="0"/>
-    <xacro:arg name="left_controller_port" default="8871"/>
-    <xacro:arg name="right_controller_ip" default="127.0.0.1"/>
-    <xacro:arg name="right_sdk_port" default="0"/>
-    <xacro:arg name="right_controller_port" default="8872"/>
+    <xacro:arg name="left_arm" default="true"/>
+    <xacro:arg name="right_arm" default="true"/>
+    <xacro:arg name="sim_gazebo" default="false"/>
+    <xacro:arg name="left_arm_ip" default="192.168.123.110"/>
+    <xacro:arg name="left_port_to_mcu" default="8881"/>
+    <xacro:arg name="left_port_to_sdk" default="8871"/>
+    <xacro:arg name="left_own_port" default="8872"/>
+    <xacro:arg name="right_arm_ip" default="192.168.123.111"/>
+    <xacro:arg name="right_port_to_mcu" default="8882"/>
+    <xacro:arg name="right_port_to_sdk" default="8873"/>
+    <xacro:arg name="right_own_port" default="8874"/>
     <!-- Include component descriptions -->
     <xacro:include filename="$(find unidingo_description)/urdf/dingo_base.xacro"/>
+    <xacro:include filename="$(find unidingo_description)/urdf/dingo_base.ros2_control.xacro"/>
     <xacro:include filename="$(find z1_description)/urdf/z1.urdf.xacro"/>
     <xacro:include filename="$(find z1_description)/urdf/z1.ros2_control.xacro"/>
@@ -41,5 +47,19 @@
     <!-- ========== Dingo Base ========== -->
     <xacro:dingo_base/>
+    <xacro:if value="$(arg sim_gazebo)">
+        <xacro:dingo_base_ros2_control/>
+        <gazebo>
+            <plugin filename="libgazebo_ros2_control.so" name="gazebo_ros2_control">
+                <parameters>$(find unidingo_description)/config/gazebo_simulation_controllers.yaml</parameters>
+                <parameters>$(find unidingo_description)/config/base_simulation_controllers.yaml</parameters>
+                <parameters>$(find unidingo_description)/config/arm_simulation_controllers.yaml</parameters>
+                <parameters>$(find unidingo_description)/config/pan_tilt_controllers.yaml</parameters>
+                <parameters>$(find unidingo_description)/config/gains_omni.yaml</parameters>
+                <parameters>$(find unidingo_description)/config/z1_gazebo_pid.yaml</parameters>
+            </plugin>
+        </gazebo>
+    </xacro:if>
     <!-- ========== Left Arm Support Pillar ========== -->
+    <xacro:if value="$(arg left_arm)">
     <link name="leftarm_link">
         <inertial>
@@ -72,4 +92,6 @@
     </joint>
     <!-- ========== Right Arm Support Pillar ========== -->
+    </xacro:if>
+    <xacro:if value="$(arg right_arm)">
     <link name="rightarm_link">
         <inertial>
@@ -101,20 +123,29 @@
         <child link="rightarm_link"/>
     </joint>
+    </xacro:if>
     <!-- ========== Left Z1 Arm ========== -->
+    <xacro:if value="$(arg left_arm)">
     <xacro:z1_arm prefix="left_" parent="leftarm_link" xyz="0 0 0" rpy="0 0 0"
                   has_gripper="$(arg has_gripper)"/>
     <xacro:z1_ros2_control prefix="left_"
-                           controller_ip="$(arg left_controller_ip)"
-                           sdk_port="$(arg left_sdk_port)"
-                           controller_port="$(arg left_controller_port)"
+                           mcu_ip="$(arg left_arm_ip)"
+                           port_to_mcu="$(arg left_port_to_mcu)"
+                           port_to_sdk="$(arg left_port_to_sdk)"
+                           own_port="$(arg left_own_port)"
+                           sim_gazebo="$(arg sim_gazebo)"
                            has_gripper="$(arg has_gripper)"/>
+    </xacro:if>
     <!-- ========== Right Z1 Arm ========== -->
+    <xacro:if value="$(arg right_arm)">
     <xacro:z1_arm prefix="right_" parent="rightarm_link" xyz="0 0 0" rpy="0 0 0"
                   has_gripper="$(arg has_gripper)"/>
     <xacro:z1_ros2_control prefix="right_"
-                           controller_ip="$(arg right_controller_ip)"
-                           sdk_port="$(arg right_sdk_port)"
-                           controller_port="$(arg right_controller_port)"
+                           mcu_ip="$(arg right_arm_ip)"
+                           port_to_mcu="$(arg right_port_to_mcu)"
+                           port_to_sdk="$(arg right_port_to_sdk)"
+                           own_port="$(arg right_own_port)"
+                           sim_gazebo="$(arg sim_gazebo)"
                            has_gripper="$(arg has_gripper)"/>
+    </xacro:if>
     <!-- ========== Pan-Tilt Head ========== -->
     <xacro:if value="$(arg pan_tilt)">
@@ -152,4 +183,21 @@
             <origin xyz="0 0 0" rpy="0 0 0"/>
         </xacro:pan_tilt>
+        <xacro:if value="$(arg sim_gazebo)">
+            <ros2_control name="pan_tilt_system" type="system">
+                <hardware>
+                    <plugin>gazebo_ros2_control/GazeboSystem</plugin>
+                </hardware>
+                <joint name="pan_tilt_yaw_joint">
+                    <command_interface name="position"/>
+                    <state_interface name="position"/>
+                    <state_interface name="velocity"/>
+                </joint>
+                <joint name="pan_tilt_pitch_joint">
+                    <command_interface name="position"/>
+                    <state_interface name="position"/>
+                    <state_interface name="velocity"/>
+                </joint>
+            </ros2_control>
+        </xacro:if>
         <!-- Camera support on top of pan-tilt -->
         <xacro:property name="camera_mount_z" value="0.1"/>

File: src/z1_ros2/z1_description/urdf/z1.ros2_control.xacro (robot description, xacro)
@@ -3,18 +3,33 @@
     <!--
       ros2_control hardware interface macro for Z1 arm.
-      @param prefix  Joint name prefix (e.g. "left_" or "right_")
-      @param controller_ip  IP address of z1_controller
-      @param sdk_port  Local UDP port (0 = auto)
-      @param controller_port  Remote UDP port of z1_controller
-      @param has_gripper  Whether this arm has a gripper
+      Z1System 保留 ROS1 风格的完整网络参数面。
+      其中 controller_ip / own_port / port_to_sdk 仍用于与 z1_ctrl_ros2 通信，
+      同时继续保留 mcu_ip / port_to_mcu 以保持与 ROS1 配置链严格一致。
+      @param mcu_ip        Arm MCU IP address
+      @param port_to_mcu   UDP port used for MCU communication
+      @param prefix        Joint name prefix (e.g. "left_" or "right_")
+      @param port_to_sdk   UDP port z1_ctrl_ros2 listens on for SDK commands
+      @param controller_ip IP address of z1_ctrl_ros2 (default: 127.0.0.1)
+      @param own_port      Local UDP port Z1System listens on for ArmState replies
+      @param has_gripper   Whether this arm has a gripper
+      @param sim_gazebo    Whether to use GazeboSystem instead of real hardware
     -->
-    <xacro:macro name="z1_ros2_control" params="prefix:='' controller_ip:='127.0.0.1' sdk_port:=0 controller_port:=8871 has_gripper:=true">
+    <xacro:macro name="z1_ros2_control" params="prefix:='' mcu_ip:='192.168.123.110' port_to_mcu:=8881 port_to_sdk:=8871 controller_ip:='127.0.0.1' own_port:=8872 has_gripper:=true sim_gazebo:=false gripper_max_tau:=10.0 gripper_epsilon:=0.01">
         <ros2_control name="${prefix}z1_system" type="system">
             <hardware>
-                <plugin>z1_hardware/Z1System</plugin>
-                <param name="controller_ip">${controller_ip}</param>
-                <param name="sdk_port">${sdk_port}</param>
-                <param name="controller_port">${controller_port}</param>
-                <param name="has_gripper">${has_gripper}</param>
+                <xacro:if value="${sim_gazebo}">
+                    <plugin>gazebo_ros2_control/GazeboSystem</plugin>
+                </xacro:if>
+                <xacro:unless value="${sim_gazebo}">
+                    <plugin>z1_hardware/Z1System</plugin>
+                    <param name="mcu_ip">${mcu_ip}</param>
+                    <param name="port_to_mcu">${port_to_mcu}</param>
+                    <param name="port_to_sdk">${port_to_sdk}</param>
+                    <param name="controller_ip">${controller_ip}</param>
+                    <param name="own_port">${own_port}</param>
+                    <param name="has_gripper">${has_gripper}</param>
+                    <param name="gripper_max_tau">${gripper_max_tau}</param>
+                    <param name="gripper_epsilon">${gripper_epsilon}</param>
+                </xacro:unless>
             </hardware>
             <joint name="${prefix}joint1">

File: src/z1_ros2/z1_description/urdf/z1_dual_standalone.urdf.xacro (robot description, xacro)
@@ -3,31 +3,37 @@
   Dual Z1 arm URDF.
   Instantiates left and right Z1 arms with separate hardware interfaces.
+  mcu_ip / port_to_mcu 已移至 z1_ctrl_ros2 节点参数，不在此处声明。
+  Z1System 只需知道如何连接各自的 z1_ctrl_ros2（port_to_sdk / own_port）。
 -->
 <robot name="z1_dual_robot" xmlns:xacro="http://www.ros.org/wiki/xacro">
-    <xacro:arg name="has_gripper" default="true"/>
-    <xacro:arg name="left_controller_ip" default="127.0.0.1"/>
-    <xacro:arg name="left_sdk_port" default="0"/>
-    <xacro:arg name="left_controller_port" default="8871"/>
-    <xacro:arg name="right_controller_ip" default="127.0.0.1"/>
-    <xacro:arg name="right_sdk_port" default="0"/>
-    <xacro:arg name="right_controller_port" default="8872"/>
+    <xacro:arg name="left_arm"            default="true"/>
+    <xacro:arg name="right_arm"           default="true"/>
+    <xacro:arg name="has_gripper"         default="true"/>
+    <xacro:arg name="left_port_to_sdk"    default="8871"/>
+    <xacro:arg name="left_own_port"       default="8872"/>
+    <xacro:arg name="right_port_to_sdk"   default="8873"/>
+    <xacro:arg name="right_own_port"      default="8874"/>
     <xacro:include filename="$(find z1_description)/urdf/z1.urdf.xacro"/>
     <xacro:include filename="$(find z1_description)/urdf/z1.ros2_control.xacro"/>
     <link name="world"/>
-    <!-- Left arm -->
+    <!-- Left arm: Z1System → z1_ctrl_ros2(left) @ 127.0.0.1:8871 -->
+    <xacro:if value="$(arg left_arm)">
     <xacro:z1_arm prefix="left_" parent="world" xyz="0 0.2 0" rpy="0 0 0"
                   has_gripper="$(arg has_gripper)"/>
     <xacro:z1_ros2_control prefix="left_"
-                           controller_ip="$(arg left_controller_ip)"
-                           sdk_port="$(arg left_sdk_port)"
-                           controller_port="$(arg left_controller_port)"
+                           port_to_sdk="$(arg left_port_to_sdk)"
+                           controller_ip="127.0.0.1"
+                           own_port="$(arg left_own_port)"
                            has_gripper="$(arg has_gripper)"/>
-    <!-- Right arm -->
+    </xacro:if>
+    <!-- Right arm: Z1System → z1_ctrl_ros2(right) @ 127.0.0.1:8873 -->
+    <xacro:if value="$(arg right_arm)">
     <xacro:z1_arm prefix="right_" parent="world" xyz="0 -0.2 0" rpy="0 0 0"
                   has_gripper="$(arg has_gripper)"/>
     <xacro:z1_ros2_control prefix="right_"
-                           controller_ip="$(arg right_controller_ip)"
-                           sdk_port="$(arg right_sdk_port)"
-                           controller_port="$(arg right_controller_port)"
+                           port_to_sdk="$(arg right_port_to_sdk)"
+                           controller_ip="127.0.0.1"
+                           own_port="$(arg right_own_port)"
                            has_gripper="$(arg has_gripper)"/>
+    </xacro:if>
 </robot>

File: src/z1_ros2/z1_description/urdf/z1_standalone.urdf.xacro (robot description, xacro)
@@ -3,10 +3,11 @@
   Standalone Z1 arm URDF for single-arm bringup.
   Instantiates one Z1 arm attached to a "world" frame.
+  mcu_ip / port_to_mcu 已移至 z1_ctrl_ros2 节点参数，不在此处声明。
+  Z1System 只需知道如何连接 z1_ctrl_ros2（controller_ip / port_to_sdk / own_port）。
 -->
 <robot name="z1_robot" xmlns:xacro="http://www.ros.org/wiki/xacro">
-    <xacro:arg name="has_gripper" default="true"/>
-    <xacro:arg name="controller_ip" default="127.0.0.1"/>
-    <xacro:arg name="sdk_port" default="0"/>
-    <xacro:arg name="controller_port" default="8871"/>
+    <xacro:arg name="has_gripper"    default="true"/>
+    <xacro:arg name="port_to_sdk"    default="8871"/>
+    <xacro:arg name="own_port"       default="8872"/>
     <xacro:include filename="$(find z1_description)/urdf/z1.urdf.xacro"/>
     <xacro:include filename="$(find z1_description)/urdf/z1.ros2_control.xacro"/>
@@ -15,7 +16,7 @@
                   has_gripper="$(arg has_gripper)"/>
     <xacro:z1_ros2_control prefix=""
-                           controller_ip="$(arg controller_ip)"
-                           sdk_port="$(arg sdk_port)"
-                           controller_port="$(arg controller_port)"
+                           port_to_sdk="$(arg port_to_sdk)"
+                           controller_ip="127.0.0.1"
+                           own_port="$(arg own_port)"
                            has_gripper="$(arg has_gripper)"/>
 </robot>
