Commit message: 文档改善/rviz改善

File: src/z1_ros/z1_description/urdf/z1_control.urdf (robot description, URDF)
Before this commit: robot z1_description, 8 links, 7 joints
Links:
- added link gripperMover, mass 0.27621302; collision mesh filename=package://z1_description/meshes/collision/z1_GripperMover.S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 scale=1 1 1; visual mesh filename=package://z1_description/meshes/visual/z1_GripperMover.dae scale=1 1 1
- added link gripperStator, mass 0.52603655; collision mesh filename=package://z1_description/meshes/collision/z1_GripperStator.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 scale=1 1 1; visual mesh filename=package://z1_description/meshes/visual/z1_GripperStator.dae scale=1 1 1
- link tool: mass 0.25 -> None; geometry 
Joints:
- added joint gripperStator: type fixed, parent link06, child gripperStator, origin xyz=0.051 0.0 0.0 rpy=0 0 0
- added joint gripper_closed_mount: type fixed, parent gripperStator, child gripperMover, origin xyz=0.049 0.0 0 rpy=0 0 0
- joint joint1: limit lower=-2.6179938779914944 upper=2.6179938779914944 effort=30.0 velocity=10 -> lower=-2.6179938779914944 upper=2.6179938779914944 effort=30.0 velocity=3.1415
- joint joint2: limit lower=0.0 upper=2.9670597283903604 effort=60.0 velocity=10 -> lower=0.0 upper=2.9670597283903604 effort=60.0 velocity=3.1415
- joint joint3: limit lower=-2.8797932657906435 upper=0.0 effort=30.0 velocity=10 -> lower=-2.8797932657906435 upper=0.0 effort=30.0 velocity=3.1415
- joint joint4: limit lower=-1.5184364492350666 upper=1.5184364492350666 effort=30.0 velocity=10 -> lower=-1.5184364492350666 upper=1.5184364492350666 effort=30.0 velocity=3.1415
- joint joint5: limit lower=-1.3439035240356338 upper=1.3439035240356338 effort=30.0 velocity=10 -> lower=-1.3439035240356338 upper=1.3439035240356338 effort=30.0 velocity=3.1415
- joint joint6: limit lower=-2.792526803190927 upper=2.792526803190927 effort=30.0 velocity=10 -> lower=-2.792526803190927 upper=2.792526803190927 effort=30.0 velocity=3.1415
